File: pcb/narfkb2.kicad_sch (KiCad schematic)
At the start: 120 parts, among them J1 MJ-4PP-9, J2 MJ-4PP-9, SW1 MX_SW_HS, SW10 MX_SW_HS, SW11 MX_SW_HS, SW12 MX_SW_HS, SW13 RotaryEncoder_Switch, SW14 MX_SW_HS, SW15 MX_SW_HS, SW16 MX_SW_HS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

Commit message: Add choc footprints
Parts:
- SW1, SW10, SW11, SW12, SW14, SW15, SW16, SW17, SW18, SW19, SW2, SW23, SW24, SW25, SW26, SW27, SW28, SW29, SW3, SW30, SW31, SW33, SW34, SW35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: footprint sepp:SW_MX_HS_1u -> sepp:SW_choc_HS_1u
