File: pcb/narfkb2.kicad_pcb (KiCad board)
At the start: 2 copper layers, 302.4 x 99.4 mm, 120 parts, among them J1 MJ-4PP-9, J2 MJ-4PP-9, SW1 MX_SW_HS, SW10 MX_SW_HS, SW11 MX_SW_HS, SW12 MX_SW_HS, SW13 RotaryEncoder_Switch, SW14 MX_SW_HS, SW15 MX_SW_HS, SW16 MX_SW_HS, SW17 MX_SW_HS, SW18 MX_SW_HS, SW19 MX_SW_HS, SW2 MX_SW_HS, SW20 actionswitch, SW21 actionswitch, SW22 actionswitch, SW23 MX_SW_HS, SW24 MX_SW_HS, SW25 MX_SW_HS, SW26 MX_SW_HS, SW27 MX_SW_HS, SW28 MX_SW_HS, SW29 MX_SW_HS, SW3 MX_SW_HS, SW30 MX_SW_HS, SW31 MX_SW_HS, SW32 RotaryEncoder_Switch, SW33 MX_SW_HS, SW34 MX_SW_HS, SW35 MX_SW_HS, SW36 MX_SW_HS, SW37 MX_SW_HS, SW38 MX_SW_HS, SW39 actionswitch, SW4 MX_SW_HS, SW40 actionswitch, SW41 actionswitch, SW42 MX_SW_HS, SW43 MX_SW_HS, SW44 MX_SW_HS, SW45 MX_SW_HS, SW46 MX_SW_HS, SW47 MX_SW_HS, SW48 MX_SW_HS, SW49 MX_SW_HS, SW5 MX_SW_HS, SW50 MX_SW_HS, SW6 MX_SW_HS, SW7 MX_SW_HS, SW8 MX_SW_HS, SW9 MX_SW_HS, U1 rp2040-zero, U2 rp2040-zero

Commit message: Add choc footprints
Parts:
- SW1, SW10, SW11, SW12, SW14, SW15, SW16, SW17, SW18, SW19, SW2, SW23, SW24, SW25, SW26, SW27, SW28, SW29, SW3, SW30, SW31, SW33, SW34, SW35, SW36, SW37, SW38, SW4, SW42, SW43, SW44, SW45, SW46, SW47, SW48, SW49, SW5, SW50, SW6, SW7, SW8, SW9: footprint sepp:SW_MX_HS_1u -> sepp:SW_choc_HS_1u
Routing:
- net L_COL6: track 46.0 -> 61.2 mm, vias 5 -> 3
- net L_COL2: track 132.1 -> 147.3 mm, vias 6 -> 5
- net L_COL4: track 88.6 -> 103.1 mm, vias 5 -> 3
- net L_COL1: track 150.0 -> 164.0 mm, vias 6 -> 4
- net R_COL6: track 66.9 -> 80.5 mm, vias 5 -> 4
- net L_COL3: track 108.0 -> 121.4 mm, vias 5 -> 4
- net R_COL5: track 86.2 -> 99.4 mm, vias 5 -> 4
- net R_COL1: track 167.6 -> 180.8 mm, vias 5 -> 4
- net R_COL3: track 124.8 -> 137.9 mm, vias 5 -> 4
- net R_COL2: track 148.4 -> 161.0 mm, vias 5 -> 4
- net R_COL4: track 107.7 -> 120.1 mm, vias 5 -> 4
- net L_COL5: track 69.6 -> 78.4 mm, vias 5 -> 3
- net L_ROW1: track 145.9 -> 153.4 mm
- net L_COL9: track 85.0 -> 90.8 mm
- net R_COL7: track 90.9 -> 96.5 mm
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
Commit message: Fix routes
Routing:
- net L_COL4: track 103.1 -> 97.3 mm
- net R_COL6: track 80.5 -> 77.0 mm, vias 4 -> 3
- net L_ROW3: track 225.9 -> 228.8 mm
- net R_COL2: track 161.0 -> 162.5 mm
- net R_COL1: track 180.8 -> 182.0 mm
- net R_ROW2: track 148.3 -> 149.5 mm
- net Net-(D50-A): track 8.21 -> 7.36 mm
- net Net-(D42-A): track 8.38 -> 7.57 mm
- net Net-(D33-A): track 8.38 -> 7.57 mm
- net Net-(D43-A): track 8.39 -> 7.57 mm
- net Net-(D34-A): track 8.39 -> 7.57 mm
- net Net-(D27-A): track 8.39 -> 7.57 mm
- net Net-(D28-A): track 8.40 -> 7.58 mm
- net Net-(D35-A): track 8.40 -> 7.58 mm
- net Net-(D44-A): track 8.40 -> 7.58 mm
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